File: HW-lab-power.sch (KiCad schematic (older format))
At the start: 16 parts, among them J1 +12V, J2 +5V, J3 +3V3, J4 GND, J5 PWR, J6 SW, J7 USB_A, SW1 SW_SPST

Commit message: Finished tweaks and setup for first revision
Parts:
- added H3, H4: MountingHole, MountingHole:MountingHole_3.2mm_M3, symbol Mechanical:MountingHole
Changed lines of the file:
@@
 	4750 3400 4750 3500
 $Comp
-L power:GND #PWR?
+L power:GND #PWR07
 U 1 1 5E17531B
 P 7450 3550
-F 0 "#PWR?" H 7450 3300 50  0001 C CNN
+F 0 "#PWR07" H 7450 3300 50  0001 C CNN
 F 1 "GND" H 7455 3377 50  0000 C CNN
 F 2 "" H 7450 3550 50  0001 C CNN
@@
 $EndComp
 $Comp
-L power:GND #PWR?
+L power:GND #PWR06
 U 1 1 5E179A17
 P 6950 3200
-F 0 "#PWR?" H 6950 2950 50  0001 C CNN
+F 0 "#PWR06" H 6950 2950 50  0001 C CNN
 F 1 "GND" H 6955 3027 50  0000 C CNN
 F 2 "" H 6950 3200 50  0001 C CNN
@@
 $EndComp
 $Comp
-L power:GND #PWR?
+L power:GND #PWR01
 U 1 1 5E179E50
 P 4450 3800
-F 0 "#PWR?" H 4450 3550 50  0001 C CNN
+F 0 "#PWR01" H 4450 3550 50  0001 C CNN
 F 1 "GND" H 4455 3627 50  0000 C CNN
 F 2 "" H 4450 3800 50  0001 C CNN
@@
 $EndComp
 $Comp
-L power:GND #PWR?
+L power:GND #PWR04
 U 1 1 5E17A3DD
 P 5500 4100
-F 0 "#PWR?" H 5500 3850 50  0001 C CNN
+F 0 "#PWR04" H 5500 3850 50  0001 C CNN
 F 1 "GND" H 5505 3927 50  0000 C CNN
 F 2 "" H 5500 4100 50  0001 C CNN
@@
 $EndComp
 $Comp
-L power:GND #PWR?
+L power:GND #PWR05
 U 1 1 5E17FA52
 P 6650 3650
-F 0 "#PWR?" H 6650 3400 50  0001 C CNN
+F 0 "#PWR05" H 6650 3400 50  0001 C CNN
 F 1 "GND" H 6655 3477 50  0000 C CNN
 F 2 "" H 6650 3650 50  0001 C CNN
@@
 $EndComp
 $Comp
-L power:GND #PWR?
+L power:GND #PWR03
 U 1 1 5E17FED7
 P 5400 3400
-F 0 "#PWR?" H 5400 3150 50  0001 C CNN
+F 0 "#PWR03" H 5400 3150 50  0001 C CNN
 F 1 "GND" H 5405 3227 50  0000 C CNN
 F 2 "" H 5400 3400 50  0001 C CNN
@@
 $EndComp
 $Comp
-L power:GND #PWR?
+L power:GND #PWR02
 U 1 1 5E180516
 P 5300 2700
-F 0 "#PWR?" H 5300 2450 50  0001 C CNN
+F 0 "#PWR02" H 5300 2450 50  0001 C CNN
 F 1 "GND" H 5305 2527 50  0000 C CNN
 F 2 "" H 5300 2700 50  0001 C CNN
@@
 Text Label 6050 3100 0    50   ~ 0
 3V3
+$Comp
+L Mechanical:MountingHole H3
+U 1 1 5E289BE2
+P 6300 4150
+F 0 "H3" H 6400 4196 50  0000 L CNN
+F 1 "MountingHole" H 6400 4105 50  0000 L CNN
+F 2 "MountingHole:MountingHole_3.2mm_M3" H 6300 4150 50  0001 C CNN
+F 3 "~" H 6300 4150 50  0001 C CNN
+	1    6300 4150
+	1    0    0    -1
+$EndComp
+$Comp
+L Mechanical:MountingHole H4
+U 1 1 5E28A5D1
+P 6300 4350
+F 0 "H4" H 6400 4396 50  0000 L CNN
+F 1 "MountingHole" H 6400 4305 50  0000 L CNN
+F 2 "MountingHole:MountingHole_3.2mm_M3" H 6300 4350 50  0001 C CNN
+F 3 "~" H 6300 4350 50  0001 C CNN
+	1    6300 4350
+	1    0    0    -1
+$EndComp
 $EndSCHEMATC
