File: HW-lab-power.kicad_pcb (KiCad board)
At the start: 2 copper layers, 85 x 85 mm, 16 parts, among them J1 +12V, J2 +5V, J3 +3V3, J4 GND, J5 PWR, J6 SW, J7 USB_A, SW1 SW_SPST

Commit message: Finished tweaks and setup for first revision
Parts:
- added H3: MountingHole, MountingHole:MountingHole_3.2mm_M3, F.Cu at (108.5, 77.5)
- added H4: MountingHole, MountingHole:MountingHole_3.2mm_M3, F.Cu at (186.5, 77.5)
- moved J7 7.50 mm to (119.6, 87.5), turned to 180 degrees
- moved D1 3.54 mm to (127.5, 70.0)
- moved D2 3.54 mm to (147.5, 70.0)
- moved D3 3.54 mm to (167.5, 70.0)
- moved H1 3.54 mm to (120.0, 132.5)
- moved H2 3.54 mm to (175.0, 132.5)
- moved J1 3.54 mm to (117.5, 70.0)
- moved J2 3.54 mm to (137.5, 70.0)
- moved J3 3.54 mm to (157.5, 70.0)
- moved J4 3.54 mm to (177.5, 70.0)
- moved J5 3.54 mm to (129.9, 90.0)
- moved J6 3.54 mm to (167.5, 92.5)
- moved R1 3.54 mm to (127.5, 72.5)
- moved R2 3.54 mm to (147.5, 72.5)
- moved R3 3.54 mm to (167.5, 72.5)
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Routing:
- net Net-(J7-Pad5): track 0.00 -> 17.0 mm
- net /5V: track 80.8 -> 89.6 mm
- net GND: track 80.1 -> 81.4 mm
Other:
- board text added: "Bench Supply Adaptor Revision 1 Thomas Bytheway"
- board text added: "USB Charger"

Commit message: Revision 1 final files
Other:
- board text added: "110W"
- board text added: "14A"
- board text added: "17A"
- board text added: "18A 216W"
- board text added: "250W"
- board text added: "Max Power"
Changed lines of the file:
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@@
   (general
     (thickness 1)
-    (drawings 76)
+    (drawings 88)
     (tracks 39)
     (zones 0)
@@
     )
   )
+  (gr_text "Max Power" (at 157.5 84) (layer F.SilkS)
+    (effects (font (size 2 2) (thickness 0.3)))
+  )
+  (gr_line (start 117.5 84) (end 133.5 84) (layer F.SilkS) (width 0.3))
+  (gr_line (start 117.5 83) (end 117.5 84) (layer F.SilkS) (width 0.3))
+  (gr_line (start 148 84) (end 141.5 84) (layer F.SilkS) (width 0.3))
+  (gr_line (start 148 80) (end 148 84) (layer F.SilkS) (width 0.3))
+  (gr_text 250W (at 137.5 84) (layer F.SilkS)
+    (effects (font (size 2 2) (thickness 0.3)))
+  )
+  (gr_line (start 144 78.5) (end 140.5 78.5) (layer F.SilkS) (width 0.3))
+  (gr_line (start 152 78.5) (end 155 78.5) (layer F.SilkS) (width 0.3))
+  (gr_text 110W (at 148 78.5) (layer F.SilkS)
+    (effects (font (size 2 2) (thickness 0.3)))
+  )
+  (gr_text "18A\n216W" (at 117.5 80) (layer F.SilkS)
+    (effects (font (size 2 2) (thickness 0.3)))
+  )
+  (gr_text 17A (at 137.5 78.5) (layer F.SilkS)
+    (effects (font (size 2 2) (thickness 0.3)))
+  )
+  (gr_text 14A (at 157.5 78.5) (layer F.SilkS)
+    (effects (font (size 2 2) (thickness 0.3)))
+  )
   (gr_line (start 157.5 90) (end 152.75 90) (layer B.Mask) (width 7))
